File: pcbIOT/pcbIOTcopybeforechange.kicad_pcb (KiCad board)
At the start: 2 copper layers, 45.9 x 38.6 mm, 34 parts, among them IC1 NRF52832-QFAA-G-R7, IC2 TPS62842DGRR, J1 Battery power in, J2 Conn_01x08_Socket, J3 Conn_01x03_Pin, J4 Conn_01x06_Socket, J5 Conn_01x06_Socket, X1 32MHz, X2 32.768kHz

Commit message: pcb bijna af
Parts:
- removed R4: 1.5kOhm, Resistor_SMD:R_0805_2012Metric_Pad1.20x1.40mm_HandSolder
- C1, C10, C11, C12, C13, C14, C15, C2, C3, C4, C5, C6, C7, C8, C9: footprint Capacitor_SMD:C_0805_2012Metric_Pad1.18x1.45mm_HandSolder -> Capacitor_SMD:C_0603_1608Metric
- R1: value 10kOhm -> 11.5kOhm; footprint Resistor_SMD:R_0805_2012Metric_Pad1.20x1.40mm_HandSolder -> Resistor_SMD:R_0603_1608Metric
- R2, R3: footprint Resistor_SMD:R_0805_2012Metric_Pad1.20x1.40mm_HandSolder -> Resistor_SMD:R_0603_1608Metric
- moved R2 2.79 mm to (141.0, 57.7)
- moved R3 2.29 mm to (141.0, 59.2)
- moved C15 1.37 mm to (123.9, 69.1)
- moved C9 1.27 mm to (142.7, 60.7)
- moved J1 1.06 mm to (127.8, 85.3)
- moved C1 1.05 mm to (126.0, 79.0)
- moved C14 0.81 mm to (123.7, 70.9)
- moved C2 0.80 mm to (123.7, 73.4)
- moved C8 0.57 mm to (142.7, 62.2)
- moved C13 0.56 mm to (138.4, 60.5)
- moved C6 0.51 mm to (137.7, 64.5)
- moved L4 0.51 mm to (142.0, 70.1)
- moved C5 0.51 mm to (128.3, 65.0)
- moved C7 0.40 mm to (132.7, 60.3)
- moved C10 0.36 mm to (144.3, 65.0)
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Connections:
- R1 pad 2: Net-(R1-Pad2) -> GND
Routing:
- net GND: track 112.1 -> 97.4 mm
- net Net-(IC1-XC2): track 15.0 -> 5.34 mm
- net Net-(IC1-P0.00/XL1): track 8.06 -> 12.3 mm
- net Net-(IC1-P0.01/XL2): track 14.2 -> 10.00 mm
- net VDD: track 127.0 -> 123.2 mm
- net SCL: track 62.1 -> 59.7 mm
- net Net-(R1-Pad2): track 2.17 -> 0.00 mm
- net Acc_int: track 36.4 -> 34.3 mm
- net Net-(IC2-EN): track 13.3 -> 11.3 mm
- net SDA: track 63.2 -> 61.7 mm
- net ToF1_INT: track 25.5 -> 24.0 mm
- net Net-(IC1-XC1): track 15.1 -> 13.8 mm
- net Net-(IC2-VSET): track 2.87 -> 1.69 mm
- net ToF1_XSHUT: track 25.7 -> 24.6 mm
- net Net-(AE1-A): track 4.56 -> 5.09 mm
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